Commit message: Imported upstream version '2.0.0' of 'upstream'

File: rotors_description/urdf/asymmetric_quadrotor.xacro (robot description, xacro)
@@ -57,18 +57,10 @@
     <xacro:insert_block name="body_inertia" />
   </xacro:multirotor_base_macro>
-    <!-- attach multirotor_base_plugin to the base_link -->
-  <gazebo>
-    <plugin filename="librotors_gazebo_multirotor_base_plugin.so" name="rosbag">
-      <robotNamespace>${namespace}</robotNamespace>
-      <linkName>base_link</linkName>
-      <rotorVelocitySlowdownSim>${rotor_velocity_slowdown_sim}</rotorVelocitySlowdownSim>
-    </plugin>
-  </gazebo>
-  <joint name="arm0_joint" type="fixed">
+  <joint name="${namespace}/arm0_joint" type="fixed">
     <origin xyz="0 0 0" rpy="0 0 0" />
-    <parent link="base_link" />
-    <child link="arm0_link" />
-  </joint>
-  <link name="arm0_link">
+    <parent link="${namespace}/base_link" />
+    <child link="${namespace}/arm0_link" />
+  </joint>
+  <link name="${namespace}/arm0_link">
     <xacro:box_inertial x="${arm_length}" y="0.03" z="0.01" mass="${(mass_rotor/3+mass_arm*5/9)*2}">
       <origin xyz="${arm_length/2} 0 0" />
@@ -87,10 +79,10 @@
     </collision>
   </link>
-  <joint name="arm1_joint" type="fixed">
+  <joint name="${namespace}/arm1_joint" type="fixed">
     <origin xyz="0 0 0" rpy="0 0 ${2*pi/3}" />
-    <parent link="base_link" />
-    <child link="arm1_link" />
-  </joint>
-  <link name="arm1_link">
+    <parent link="${namespace}/base_link" />
+    <child link="${namespace}/arm1_link" />
+  </joint>
+  <link name="${namespace}/arm1_link">
     <xacro:box_inertial x="${arm_length}" y="0.03" z="0.01" mass="${mass_arm}">
       <origin xyz="${arm_length/2} 0 0" />
@@ -109,10 +101,10 @@
     </collision>
   </link>
-  <joint name="arm2_joint" type="fixed">
+  <joint name="${namespace}/arm2_joint" type="fixed">
     <origin xyz="0 0 0" rpy="0 0 ${pi}" />
-    <parent link="base_link" />
-    <child link="arm2_link" />
-  </joint>
-  <link name="arm2_link">
+    <parent link="${namespace}/base_link" />
+    <child link="${namespace}/arm2_link" />
+  </joint>
+  <link name="${namespace}/arm2_link">
     <xacro:box_inertial x="${arm_length/3}" y="0.03" z="0.01" mass="${mass_arm/3}">
       <origin xyz="${arm_length/6} 0 0" />
@@ -131,10 +123,10 @@
     </collision>
   </link>
-  <joint name="arm3_joint" type="fixed">
+  <joint name="${namespace}/arm3_joint" type="fixed">
     <origin xyz="0 0 0" rpy="0 0 -${2*pi/3}" />
-    <parent link="base_link" />
-    <child link="arm3_link" />
-  </joint>
-  <link name="arm3_link">
+    <parent link="${namespace}/base_link" />
+    <child link="${namespace}/arm3_link" />
+  </joint>
+  <link name="${namespace}/arm3_link">
     <xacro:box_inertial x="${arm_length}" y="0.03" z="0.01" mass="${mass_arm}">
       <origin xyz="${arm_length/2} 0 0" />
@@ -160,5 +152,5 @@
     motor_constant="${motor_constant}"
     moment_constant="${moment_constant}"
-    parent="arm0_link"
+    parent="${namespace}/arm0_link"
     mass_rotor="${mass_rotor}"
     radius_rotor="${radius_rotor}"
@@ -169,5 +161,7 @@
     rotor_drag_coefficient="${rotor_drag_coefficient}"
     rolling_moment_coefficient="${rolling_moment_coefficient}"
-    color="Red">
+    color="Red"
+    use_own_mesh="false"
+    mesh="">
     <origin xyz="${arm_length} 0 ${rotor_offset_top}" rpy="0 0 0" />
     <xacro:insert_block name="rotor_inertia" />
@@ -179,5 +173,5 @@
     motor_constant="${motor_constant}"
     moment_constant="${moment_constant}"
-    parent="arm1_link"
+    parent="${namespace}/arm1_link"
     mass_rotor="${mass_rotor}"
     radius_rotor="${radius_rotor}"
@@ -188,5 +182,7 @@
     rotor_drag_coefficient="${rotor_drag_coefficient}"
     rolling_moment_coefficient="${rolling_moment_coefficient}"
-    color="Blue">
+    color="Blue"
+    use_own_mesh="false"
+    mesh="">
     <origin xyz="${arm_length} 0 ${rotor_offset_top}" rpy="0 0 0" />
     <xacro:insert_block name="rotor_inertia" />
@@ -198,5 +194,5 @@
     motor_constant="${motor_constant}"
     moment_constant="${moment_constant}"
-    parent="arm2_link"
+    parent="${namespace}/arm2_link"
     mass_rotor="${mass_rotor}"
     radius_rotor="${radius_rotor}"
@@ -207,5 +203,7 @@
     rotor_drag_coefficient="${rotor_drag_coefficient}"
     rolling_moment_coefficient="${rolling_moment_coefficient}"
-    color="Yellow">
+    color="Yellow"
+    use_own_mesh="false"
+    mesh="">
     <origin xyz="${arm_length/3} 0 ${rotor_offset_top}" rpy="0 0 0" />
     <xacro:insert_block name="rotor_inertia" />
@@ -217,5 +215,5 @@
     motor_constant="${motor_constant}"
     moment_constant="${moment_constant}"
-    parent="arm3_link"
+    parent="${namespace}/arm3_link"
     mass_rotor="${mass_rotor}"
     radius_rotor="${radius_rotor}"
@@ -226,5 +224,7 @@
     rotor_drag_coefficient="${rotor_drag_coefficient}"
     rolling_moment_coefficient="${rolling_moment_coefficient}"
-    color="Blue">
+    color="Blue"
+    use_own_mesh="false"
+    mesh="">
     <origin xyz="${arm_length} 0 ${rotor_offset_top}" rpy="0 0 0" />
     <xacro:insert_block name="rotor_inertia" />

File: rotors_description/urdf/asymmetric_quadrotor_base.xacro (robot description, xacro)
@@ -23,7 +23,7 @@
   <xacro:controller_plugin_macro namespace="${namespace}" imu_sub_topic="imu" />
   <!-- Mount an ADIS16448 IMU. -->
-  <xacro:default_imu namespace="${namespace}" />
+  <xacro:default_imu namespace="${namespace}" parent_link="${namespace}/base_link" />
   <xacro:if value="$(arg enable_ground_truth)">
-    <xacro:ground_truth_imu_and_odometry namespace="${namespace}" />
+    <xacro:ground_truth_imu_and_odometry namespace="${namespace}" parent_link="${namespace}/base_link" />
   </xacro:if>
   <xacro:if value="$(arg enable_logging)">

File: rotors_description/urdf/component_snippets.xacro (robot description, xacro)
@@ -25,6 +25,6 @@
         <robotNamespace>${namespace}</robotNamespace>
         <bagFileName>${bag_file}</bagFileName>
-        <linkName>base_link</linkName>
-        <frameId>base_link</frameId>
+        <linkName>${namespace}/base_link</linkName>
+        <frameId>${namespace}/base_link</frameId>
         <commandAttitudeThrustSubTopic>command/attitude</commandAttitudeThrustSubTopic>
         <commandAttitudeThrustPubTopic>command/attitude</commandAttitudeThrustPubTopic>
@@ -47,5 +47,5 @@
       <xacro:if value="${enable_visual}">
         <visual>
-          <origin xyz="0 0 0" rpy="0 0 0" />
+          <origin xyz="0 0 0" rpy="0 ${pi/2} 0" />
           <geometry>
             <xacro:insert_block name="geometry" />
@@ -336,6 +336,6 @@
     <gazebo>
       <plugin filename="librotors_gazebo_wind_plugin.so" name="wind_plugin">
-        <frameId>base_link</frameId>
-        <linkName>base_link</linkName>
+        <frameId>world</frameId>
+        <linkName>${namespace}/base_link</linkName>
         <robotNamespace>${namespace}</robotNamespace>
         <xyzOffset>${xyz_offset}</xyzOffset> <!-- [m] [m] [m] -->
@@ -366,6 +366,6 @@
       noise_mean="0.0"
       noise_stddev="0.007"
-      enable_visual="false">
-      <cylinder length="0.01" radius="0.007" />
+      enable_visual="true">
+      <mesh filename="package://rotors_description/meshes/vi_camera.dae" scale="1 1 1" />
       <xacro:insert_block name="origin" />
     </xacro:camera_macro>
@@ -558,10 +558,10 @@
     </xacro:imu_plugin_macro>
   </xacro:macro>
-  <xacro:macro name="ground_truth_imu_and_odometry" params="namespace">
+  <xacro:macro name="ground_truth_imu_and_odometry" params="namespace parent_link">
     <!-- Mount an IMU providing ground truth. -->
     <xacro:imu_plugin_macro
       namespace="${namespace}"
       imu_suffix="gt"
-      parent_link="base_link"
+      parent_link="${parent_link}"
       imu_topic="ground_truth/imu"
       mass_imu_sensor="0.00001"
@@ -581,5 +581,5 @@
       namespace="${namespace}/ground_truth"
       odometry_sensor_suffix="gt"
-      parent_link="base_link"
+      parent_link="${parent_link}"
       pose_topic="pose"
       pose_with_covariance_topic="pose_with_covariance"
@@ -607,10 +607,10 @@
     </xacro:odometry_plugin_macro>
   </xacro:macro>
-  <xacro:macro name="default_imu" params="namespace">
+  <xacro:macro name="default_imu" params="namespace parent_link">
     <!-- ADIS16448 IMU. -->
     <xacro:imu_plugin_macro
       namespace="${namespace}"
       imu_suffix=""
-      parent_link="base_link"
+      parent_link="${parent_link}"
       imu_topic="imu"
       mass_imu_sensor="0.015"

File: rotors_description/urdf/firefly.xacro (robot description, xacro)
@@ -21,5 +21,5 @@
   <xacro:property name="rotor_velocity_slowdown_sim" value="10" />
   <xacro:property name="use_mesh_file" value="true" />
-  <xacro:property name="mesh_file" value="firefly.dae" />
+  <xacro:property name="mesh_file" value="package://rotors_description/meshes/firefly.dae" />
   <xacro:property name="mass" value="1.5" /> <!-- [kg] -->
   <xacro:property name="body_width" value="0.1" /> <!-- [m] -->
@@ -66,5 +66,5 @@
     motor_constant="${motor_constant}"
     moment_constant="${moment_constant}"
-    parent="base_link"
+    parent="${namespace}/base_link"
     mass_rotor="${mass_rotor}"
     radius_rotor="${radius_rotor}"
@@ -75,5 +75,7 @@
     rotor_drag_coefficient="${rotor_drag_coefficient}"
     rolling_moment_coefficient="${rolling_moment_coefficient}"
-    color="Red">
+    color="Red"
+    use_own_mesh="false"
+    mesh="">
     <origin xyz="${cos30*arm_length} ${sin30*arm_length} ${rotor_offset_top}" rpy="0 0 0" />
     <xacro:insert_block name="rotor_inertia" />
@@ -85,5 +87,5 @@
     motor_constant="${motor_constant}"
     moment_constant="${moment_constant}"
-    parent="base_link"
+    parent="${namespace}/base_link"
     mass_rotor="${mass_rotor}"
     radius_rotor="${radius_rotor}"
@@ -94,5 +96,7 @@
     rotor_drag_coefficient="${rotor_drag_coefficient}"
     rolling_moment_coefficient="${rolling_moment_coefficient}"
-    color="Blue">
+    color="Blue"
+    use_own_mesh="false"
+    mesh="">
     <origin xyz="0 ${arm_length} ${rotor_offset_top}" rpy="0 0 0" />
     <xacro:insert_block name="rotor_inertia" />
@@ -103,5 +107,5 @@
     motor_constant="${motor_constant}"
     moment_constant="${moment_constant}"
-    parent="base_link"
+    parent="${namespace}/base_link"
     mass_rotor="${mass_rotor}"
     radius_rotor="${radius_rotor}"
@@ -112,5 +116,7 @@
     rotor_drag_coefficient="${rotor_drag_coefficient}"
     rolling_moment_coefficient="${rolling_moment_coefficient}"
-    color="Blue">
+    color="Blue"
+    use_own_mesh="false"
+    mesh="">
     <origin xyz="-${cos30*arm_length} ${sin30*arm_length} ${rotor_offset_top}" rpy="0 0 0" />
     <xacro:insert_block name="rotor_inertia" />
@@ -121,5 +127,5 @@
     motor_constant="${motor_constant}"
     moment_constant="${moment_constant}"
-    parent="base_link"
+    parent="${namespace}/base_link"
     mass_rotor="${mass_rotor}"
     radius_rotor="${radius_rotor}"
@@ -130,5 +136,7 @@
     rotor_drag_coefficient="${rotor_drag_coefficient}"
     rolling_moment_coefficient="${rolling_moment_coefficient}"
-    color="Blue">
+    color="Blue"
+    use_own_mesh="false"
+    mesh="">
     <origin xyz="-${cos30*arm_length} -${sin30*arm_length} ${rotor_offset_top}" rpy="0 0 0" />
     <xacro:insert_block name="rotor_inertia" />
@@ -140,5 +148,5 @@
     motor_constant="${motor_constant}"
     moment_constant="${moment_constant}"
-    parent="base_link"
+    parent="${namespace}/base_link"
     mass_rotor="${mass_rotor}"
     radius_rotor="${radius_rotor}"
@@ -149,5 +157,7 @@
     rotor_drag_coefficient="${rotor_drag_coefficient}"
     rolling_moment_coefficient="${rolling_moment_coefficient}"
-    color="Blue">
+    color="Blue"
+    use_own_mesh="false"
+    mesh="">
     <origin xyz="0 -${arm_length} ${rotor_offset_top}" rpy="0 0 0" />
     <xacro:insert_block name="rotor_inertia" />
@@ -159,5 +169,5 @@
     motor_constant="${motor_constant}"
     moment_constant="${moment_constant}"
-    parent="base_link"
+    parent="${namespace}/base_link"
     mass_rotor="${mass_rotor}"
     radius_rotor="${radius_rotor}"
@@ -168,5 +178,7 @@
     rotor_drag_coefficient="${rotor_drag_coefficient}"
     rolling_moment_coefficient="${rolling_moment_coefficient}"
-    color="Red">
+    color="Red"
+    use_own_mesh="false"
+    mesh="">
     <origin xyz="${cos30*arm_length} -${sin30*arm_length} ${rotor_offset_top}" rpy="0 0 0" />
     <xacro:insert_block name="rotor_inertia" />

File: rotors_description/urdf/firefly_base.xacro (robot description, xacro)
@@ -23,7 +23,7 @@
   <xacro:controller_plugin_macro namespace="${namespace}" imu_sub_topic="imu" />
   <!-- Mount an ADIS16448 IMU. -->
-  <xacro:default_imu namespace="${namespace}" />
+  <xacro:default_imu namespace="${namespace}" parent_link="${namespace}/base_link" />
   <xacro:if value="$(arg enable_ground_truth)">
-    <xacro:ground_truth_imu_and_odometry namespace="${namespace}" />
+    <xacro:ground_truth_imu_and_odometry namespace="${namespace}" parent_link="${namespace}/base_link" />
   </xacro:if>
   <xacro:if value="$(arg enable_logging)">

File: rotors_description/urdf/hummingbird.xacro (robot description, xacro)
@@ -22,5 +22,5 @@
   <xacro:property name="rotor_velocity_slowdown_sim" value="10" />
   <xacro:property name="use_mesh_file" value="true" />
-  <xacro:property name="mesh_file" value="hummingbird.dae" />
+  <xacro:property name="mesh_file" value="package://rotors_description/meshes/hummingbird.dae" />
   <xacro:property name="mass" value="0.68" /> <!-- [kg] -->
   <xacro:property name="body_width" value="0.1" /> <!-- [m] -->
@@ -64,5 +64,5 @@
     motor_constant="${motor_constant}"
     moment_constant="${moment_constant}"
-    parent="base_link"
+    parent="${namespace}/base_link"
     mass_rotor="${mass_rotor}"
     radius_rotor="${radius_rotor}"
@@ -73,5 +73,7 @@
     rotor_drag_coefficient="${rotor_drag_coefficient}"
     rolling_moment_coefficient="${rolling_moment_coefficient}"
-    color="Red">
+    color="Red"
+    use_own_mesh="false"
+    mesh="">
     <origin xyz="${arm_length} 0 ${rotor_offset_top}" rpy="0 0 0" />
     <xacro:insert_block name="rotor_inertia" />
@@ -83,5 +85,5 @@
     motor_constant="${motor_constant}"
     moment_constant="${moment_constant}"
-    parent="base_link"
+    parent="${namespace}/base_link"
     mass_rotor="${mass_rotor}"
     radius_rotor="${radius_rotor}"
@@ -92,5 +94,7 @@
     rotor_drag_coefficient="${rotor_drag_coefficient}"
     rolling_moment_coefficient="${rolling_moment_coefficient}"
-    color="Blue">
+    color="Blue"
+    use_own_mesh="false"
+    mesh="">
     <origin xyz="0 ${arm_length} ${rotor_offset_top}" rpy="0 0 0" />
     <xacro:insert_block name="rotor_inertia" />
@@ -102,5 +106,5 @@
     motor_constant="${motor_constant}"
     moment_constant="${moment_constant}"
-    parent="base_link"
+    parent="${namespace}/base_link"
     mass_rotor="${mass_rotor}"
     radius_rotor="${radius_rotor}"
@@ -111,5 +115,7 @@
     rotor_drag_coefficient="${rotor_drag_coefficient}"
     rolling_moment_coefficient="${rolling_moment_coefficient}"
-    color="Blue">
+    color="Blue"
+    use_own_mesh="false"
+    mesh="">
     <origin xyz="-${arm_length} 0 ${rotor_offset_top}" rpy="0 0 0" />
     <xacro:insert_block name="rotor_inertia" />
@@ -121,5 +127,5 @@
     motor_constant="${motor_constant}"
     moment_constant="${moment_constant}"
-    parent="base_link"
+    parent="${namespace}/base_link"
     mass_rotor="${mass_rotor}"
     radius_rotor="${radius_rotor}"
@@ -130,5 +136,7 @@
     rotor_drag_coefficient="${rotor_drag_coefficient}"
     rolling_moment_coefficient="${rolling_moment_coefficient}"
-    color="Blue">
+    color="Blue"
+    use_own_mesh="false"
+    mesh="">
     <origin xyz="0 -${arm_length} ${rotor_offset_top}" rpy="0 0 0" />
     <xacro:insert_block name="rotor_inertia" />

File: rotors_description/urdf/hummingbird_base.xacro (robot description, xacro)
@@ -23,7 +23,7 @@
   <xacro:controller_plugin_macro namespace="${namespace}" imu_sub_topic="imu" />
   <!-- Mount an ADIS16448 IMU. -->
-  <xacro:default_imu namespace="${namespace}" />
+  <xacro:default_imu namespace="${namespace}" parent_link="${namespace}/base_link" />
   <xacro:if value="$(arg enable_ground_truth)">
-    <xacro:ground_truth_imu_and_odometry namespace="${namespace}" />
+    <xacro:ground_truth_imu_and_odometry namespace="${namespace}" parent_link="${namespace}/base_link" />
   </xacro:if>
   <xacro:if value="$(arg enable_logging)">

File: rotors_description/urdf/multirotor_base.xacro (robot description, xacro)
@@ -34,11 +34,11 @@
   <xacro:macro name="multirotor_base_macro"
     params="robot_namespace mass body_width body_height use_mesh_file mesh_file *inertia">
-    <link name="base_link"></link>
-    <joint name="base_joint" type="fixed">
+    <link name="${robot_namespace}/base_link"></link>
+    <joint name="${robot_namespace}/base_joint" type="fixed">
       <origin xyz="0 0 0" rpy="0 0 0" />
-      <parent link="base_link" />
-      <child link="base_link_inertia" />
+      <parent link="${robot_namespace}/base_link" />
+      <child link="${robot_namespace}/base_link_inertia" />
     </joint>
-    <link name="base_link_inertia">
+    <link name="${robot_namespace}/base_link_inertia">
       <inertial>
         <mass value="${mass}" />  <!-- [kg] -->
@@ -50,6 +50,5 @@
         <geometry>
           <xacro:if value="${use_mesh_file}">
-            <mesh filename="package://rotors_description/meshes/${mesh_file}"
-              scale="1 1 1" />
+            <mesh filename="${mesh_file}" scale="1 1 1" />
           </xacro:if>
           <xacro:unless value="${use_mesh_file}">
@@ -69,5 +68,5 @@
       <plugin filename="librotors_gazebo_multirotor_base_plugin.so" name="rosbag">
         <robotNamespace>${robot_namespace}</robotNamespace>
-        <linkName>base_link</linkName>
+        <linkName>${robot_namespace}/base_link</linkName>
         <rotorVelocitySlowdownSim>${rotor_velocity_slowdown_sim}</rotorVelocitySlowdownSim>
       </plugin>
@@ -76,12 +75,12 @@
   <!-- Rotor joint and link -->
   <xacro:macro name="vertical_rotor"
-    params="robot_namespace suffix direction motor_constant moment_constant parent mass_rotor radius_rotor time_constant_up time_constant_down max_rot_velocity motor_number rotor_drag_coefficient rolling_moment_coefficient color *origin *inertia">
-    <joint name="rotor_${motor_number}_joint" type="continuous">
+    params="robot_namespace suffix direction motor_constant moment_constant parent mass_rotor radius_rotor time_constant_up time_constant_down max_rot_velocity motor_number rotor_drag_coefficient rolling_moment_coefficient color use_own_mesh mesh *origin *inertia">
+    <joint name="${robot_namespace}/rotor_${motor_number}_joint" type="continuous">
       <xacro:insert_block name="origin" />
       <axis xyz="0 0 1" />
       <parent link="${parent}" />
-      <child link="rotor_${motor_number}" />
+      <child link="${robot_namespace}/rotor_${motor_number}" />
     </joint>
-    <link name="rotor_${motor_number}">
+    <link name="${robot_namespace}/rotor_${motor_number}">
       <inertial>
         <mass value="${mass_rotor}" /> <!-- [kg] -->
@@ -91,7 +90,13 @@
         <geometry>
           <!-- <cylinder length="0.005" radius="${radius_rotor}"/> --> <!-- [m] -->
-          <mesh filename="package://rotors_description/meshes/propeller_${direction}.dae"
-            scale="${radius_rotor} ${radius_rotor} ${radius_rotor}" /> <!-- The propeller meshes have a radius of 1m -->
-          <!-- <box size="${2*radius_rotor} 0.01 0.005"/> -->
+          <xacro:if value="${use_own_mesh}">
+            <mesh filename="${mesh}"
+              scale="1 1 1" />
+          </xacro:if>
+          <xacro:unless value="${use_own_mesh}">
+            <mesh filename="package://rotors_description/meshes/propeller_${direction}.dae"
+              scale="${radius_rotor} ${radius_rotor} ${radius_rotor}" /> <!-- The propeller meshes have a radius of 1m -->
+            <!-- <box size="${2*radius_rotor} 0.01 0.005"/> -->
+          </xacro:unless>
         </geometry>
       </visual>
@@ -103,8 +108,8 @@
     </link>
     <gazebo>
-      <plugin name="${suffix}_motor_model" filename="librotors_gazebo_motor_model.so">
+      <plugin name="${robot_namespace}_${suffix}_motor_model" filename="librotors_gazebo_motor_model.so">
         <robotNamespace>${robot_namespace}</robotNamespace>
-        <jointName>rotor_${motor_number}_joint</jointName>
-        <linkName>rotor_${motor_number}</linkName>
+        <jointName>${robot_namespace}/rotor_${motor_number}_joint</jointName>
+        <linkName>${robot_namespace}/rotor_${motor_number}</linkName>
         <turningDirection>${direction}</turningDirection>
         <timeConstantUp>${time_constant_up}</timeConstantUp>
@@ -121,5 +126,5 @@
       </plugin>
     </gazebo>
-    <gazebo reference="rotor_${motor_number}">
+    <gazebo reference="${robot_namespace}/rotor_${motor_number}">
       <material>Gazebo/${color}</material>
     </gazebo>
